File: kicad_102.sch (KiCad schematic (older format))
At the start: 6 parts, among them U1 NE555

Commit message: components associated
Parts:
- C1: footprint (none) -> Capacitors_SMD:C_0603_HandSoldering
- D1: footprint (none) -> LEDs:LED-8MM
- R1, R2, R3: footprint (none) -> Resistors_ThroughHole:Resistor_Horizontal_RM10mm
Changed lines of the file:
@@
 LIBS:contrib
 LIBS:valves
-LIBS:temp-cache
+LIBS:kicad_102-cache
 EELAYER 25 0
 EELAYER END
@@
 F 0 "R2" V 4880 4250 50  0000 C CNN
 F 1 "1k" V 4800 4250 50  0000 C CNN
-F 2 "" V 4730 4250 50  0000 C CNN
+F 2 "Resistors_ThroughHole:Resistor_Horizontal_RM10mm" V 4730 4250 50  0001 C CNN
 F 3 "" H 4800 4250 50  0000 C CNN
 	1    4800 4250
@@
 F 0 "R1" V 4880 3800 50  0000 C CNN
 F 1 "447" V 4800 3800 50  0000 C CNN
-F 2 "" V 4730 3800 50  0000 C CNN
+F 2 "Resistors_ThroughHole:Resistor_Horizontal_RM10mm" V 4730 3800 50  0001 C CNN
 F 3 "" H 4800 3800 50  0000 C CNN
 	1    4800 3800
@@
 F 0 "R3" V 4530 4800 50  0000 C CNN
 F 1 "1k" V 4450 4800 50  0000 C CNN
-F 2 "" V 4380 4800 50  0000 C CNN
+F 2 "Resistors_ThroughHole:Resistor_Horizontal_RM10mm" V 4380 4800 50  0001 C CNN
 F 3 "" H 4450 4800 50  0000 C CNN
 	1    4450 4800
@@
 F 0 "C1" H 2675 4750 50  0000 L CNN
 F 1 "1uF" H 2675 4550 50  0000 L CNN
-F 2 "" H 2688 4500 50  0000 C CNN
+F 2 "Capacitors_SMD:C_0603_HandSoldering" H 2688 4500 50  0001 C CNN
 F 3 "" H 2650 4650 50  0000 C CNN
 	1    2650 4650
@@
 $EndComp
 $Comp
-L VCC #PWR1
+L VCC #PWR01
 U 1 1 5811472F
 P 3750 3550
-F 0 "#PWR1" H 3750 3400 50  0001 C CNN
+F 0 "#PWR01" H 3750 3400 50  0001 C CNN
 F 1 "VCC" H 3750 3700 50  0000 C CNN
 F 2 "" H 3750 3550 50  0000 C CNN
@@
 F 0 "D1" H 4450 5250 50  0000 C CNN
 F 1 "LED" H 4450 5050 50  0000 C CNN
-F 2 "" H 4450 5150 50  0000 C CNN
+F 2 "LEDs:LED-8MM" H 4450 5150 50  0001 C CNN
 F 3 "" H 4450 5150 50  0000 C CNN
 	1    4450 5150
@@
 Connection ~ 3750 5350
 $Comp
-L GND #PWR2
+L GND #PWR02
 U 1 1 581153C1
 P 3750 5450
-F 0 "#PWR2" H 3750 5200 50  0001 C CNN
+F 0 "#PWR02" H 3750 5200 50  0001 C CNN
 F 1 "GND" H 3750 5300 50  0000 C CNN
 F 2 "" H 3750 5450 50  0000 C CNN
