File: kicad_102.kicad_pcb (KiCad board)
At the start: 2 copper layers, 6 parts, among them U1 NE555

Commit message: pcb finished
Parts:
- C1: moved to B.Cu
- moved R1 7.62 mm to (192.4, 119.4)
- moved R3 2.54 mm to (177.2, 127.0)
Routing:
- net Net-(R1-Pad2): track 0.00 -> 38.7 mm
- net VCC: track 0.00 -> 36.3 mm, vias 0 -> 2
- net Net-(D1-Pad2): track 0.00 -> 25.3 mm, vias 0 -> 2
- net Net-(C1-Pad1): track 0.00 -> 19.5 mm
- net GND: track 0.00 -> 16.1 mm
- net Net-(R3-Pad1): track 0.00 -> 12.7 mm
Other:
- board outline added: 29.8 x 34.3 mm
Changed lines of the file:
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@@
   (general
     (links 11)
-    (no_connects 11)
-    (area 0 0 0 0)
+    (no_connects 0)
+    (area 167.60988 97.03 196.98012 131.885)
     (thickness 1.6)
-    (drawings 0)
-    (tracks 0)
+    (drawings 4)
+    (tracks 40)
     (zones 0)
     (modules 6)
@@
     (pad_to_mask_clearance 0.2)
     (aux_axis_origin 0 0)
+    (grid_origin 186.055 112.395)
     (visible_elements FFFFFF7F)
     (pcbplotparams
@@
     (add_net VCC)
   )
-  (module Capacitors_SMD:C_0603_HandSoldering (layer F.Cu)
+  (module Capacitors_SMD:C_0603_HandSoldering (layer B.Cu)
     (at 172.72 113.665 90)
     (descr "Capacitor SMD 0603, hand soldering")
     (tags "capacitor 0603")
     (attr smd)
-    (fp_text reference C1 (at 0 -1.9 90) (layer F.SilkS)
-      (effects (font (size 1 1) (thickness 0.15)))
-    )
-    (fp_text value 1uF (at 0 1.9 90) (layer F.Fab)
-      (effects (font (size 1 1) (thickness 0.15)))
-    )
-    (fp_line (start -0.8 0.4) (end -0.8 -0.4) (layer F.Fab) (width 0.15))
-    (fp_line (start 0.8 0.4) (end -0.8 0.4) (layer F.Fab) (width 0.15))
-    (fp_line (start 0.8 -0.4) (end 0.8 0.4) (layer F.Fab) (width 0.15))
-    (fp_line (start -0.8 -0.4) (end 0.8 -0.4) (layer F.Fab) (width 0.15))
-    (fp_line (start -1.85 -0.75) (end 1.85 -0.75) (layer F.CrtYd) (width 0.05))
-    (fp_line (start -1.85 0.75) (end 1.85 0.75) (layer F.CrtYd) (width 0.05))
-    (fp_line (start -1.85 -0.75) (end -1.85 0.75) (layer F.CrtYd) (width 0.05))
-    (fp_line (start 1.85 -0.75) (end 1.85 0.75) (layer F.CrtYd) (width 0.05))
-    (fp_line (start -0.35 -0.6) (end 0.35 -0.6) (layer F.SilkS) (width 0.15))
-    (fp_line (start 0.35 0.6) (end -0.35 0.6) (layer F.SilkS) (width 0.15))
-    (pad 1 smd rect (at -0.95 0 90) (size 1.2 0.75) (layers F.Cu F.Paste F.Mask)
+    (fp_text reference C1 (at 0 1.9 90) (layer B.SilkS)
+      (effects (font (size 1 1) (thickness 0.15)) (justify mirror))
+    )
+    (fp_text value 1uF (at 0 -1.9 90) (layer B.Fab)
+      (effects (font (size 1 1) (thickness 0.15)) (justify mirror))
+    )
+    (fp_line (start -0.8 -0.4) (end -0.8 0.4) (layer B.Fab) (width 0.15))
+    (fp_line (start 0.8 -0.4) (end -0.8 -0.4) (layer B.Fab) (width 0.15))
+    (fp_line (start 0.8 0.4) (end 0.8 -0.4) (layer B.Fab) (width 0.15))
+    (fp_line (start -0.8 0.4) (end 0.8 0.4) (layer B.Fab) (width 0.15))
+    (fp_line (start -1.85 0.75) (end 1.85 0.75) (layer B.CrtYd) (width 0.05))
+    (fp_line (start -1.85 -0.75) (end 1.85 -0.75) (layer B.CrtYd) (width 0.05))
+    (fp_line (start -1.85 0.75) (end -1.85 -0.75) (layer B.CrtYd) (width 0.05))
+    (fp_line (start 1.85 0.75) (end 1.85 -0.75) (layer B.CrtYd) (width 0.05))
+    (fp_line (start -0.35 0.6) (end 0.35 0.6) (layer B.SilkS) (width 0.15))
+    (fp_line (start 0.35 -0.6) (end -0.35 -0.6) (layer B.SilkS) (width 0.15))
+    (pad 1 smd rect (at -0.95 0 90) (size 1.2 0.75) (layers B.Cu B.Paste B.Mask)
       (net 1 "Net-(C1-Pad1)"))
-    (pad 2 smd rect (at 0.95 0 90) (size 1.2 0.75) (layers F.Cu F.Paste F.Mask)
+    (pad 2 smd rect (at 0.95 0 90) (size 1.2 0.75) (layers B.Cu B.Paste B.Mask)
       (net 2 GND))
     (model Capacitors_SMD.3dshapes/C_0603_HandSoldering.wrl
@@
   )
   (module Resistors_ThroughHole:Resistor_Horizontal_RM10mm (layer F.Cu)
-    (at 192.405 111.76 270)
+    (at 192.405 119.38 270)
     (descr "Resistor, Axial,  RM 10mm, 1/3W")
     (tags "Resistor Axial RM 10mm 1/3W")
@@
   )
   (module Resistors_ThroughHole:Resistor_Horizontal_RM10mm (layer F.Cu)
-    (at 177.165 129.54)
+    (at 177.165 127)
     (descr "Resistor, Axial,  RM 10mm, 1/3W")
     (tags "Resistor Axial RM 10mm 1/3W")
@@
     )
   )
+  (gr_line (start 196.85 131.445) (end 167.005 131.445) (angle 90) (layer Edge.Cuts) (width 0.15))
+  (gr_line (start 196.85 97.155) (end 196.85 131.445) (angle 90) (layer Edge.Cuts) (width 0.15))
+  (gr_line (start 167.005 97.155) (end 196.85 97.155) (angle 90) (layer Edge.Cuts) (width 0.15))
+  (gr_line (start 167.005 131.445) (end 167.005 97.155) (angle 90) (layer Edge.Cuts) (width 0.15))
+  (segment (start 178.435 114.935) (end 180.34 114.935) (width 0.25) (layer B.Cu) (net 1) (status 400000))
+  (segment (start 182.88 117.475) (end 186.055 117.475) (width 0.25) (layer B.Cu) (net 1) (status 800000))
+  (segment (start 180.34 114.935) (end 182.88 117.475) (width 0.25) (layer B.Cu) (net 1))
+  (segment (start 172.085 119.38) (end 172.085 115.25) (width 0.25) (layer B.Cu) (net 1))
+  (segment (start 172.085 115.25) (end 172.72 114.615) (width 0.25) (layer B.Cu) (net 1))
+  (segment (start 178.435 114.935) (end 173.04 114.935) (width 0.25) (layer B.Cu) (net 1))
+  (segment (start 173.04 114.935) (end 172.72 114.615) (width 0.25) (layer B.Cu) (net 1))
+  (segment (start 178.435 112.395) (end 181.61 109.22) (width 0.25) (layer B.Cu) (net 2))
+  (segment (start 181.61 109.22) (end 181.61 103.505) (width 0.25) (layer B.Cu) (net 2))
+  (segment (start 172.72 112.715) (end 178.115 112.715) (width 0.25) (layer B.Cu) (net 2))
+  (segment (start 178.115 112.715) (end 178.435 112.395) (width 0.25) (layer B.Cu) (net 2))
+  (segment (start 187.325 127) (end 187.325 125.73) (width 0.25) (layer B.Cu) (net 3) (status 400000))
+  (segment (start 184.15 106.68) (end 184.15 103.505) (width 0.25) (layer B.Cu) (net 3) (status 800000))
+  (segment (start 187.96 110.49) (end 184.15 106.68) (width 0.25) (layer B.Cu) (net 3))
+  (via (at 187.96 110.49) (size 0.6) (drill 0.4) (layers F.Cu B.Cu) (net 3))
+  (segment (start 187.96 117.475) (end 187.96 110.49) (width 0.25) (layer F.Cu) (net 3))
+  (via (at 187.96 117.475) (size 0.6) (drill 0.4) (layers F.Cu B.Cu) (net 3))
+  (segment (start 187.96 125.095) (end 187.96 117.475) (width 0.25) (layer B.Cu) (net 3))
+  (segment (start 187.325 125.73) (end 187.96 125.095) (width 0.25) (layer B.Cu) (net 3))
+  (segment (start 178.435 120.015) (end 182.245 120.015) (width 0.25) (layer B.Cu) (net 4) (status 400000))
+  (segment (start 192.405 120.65) (end 192.405 119.38) (width 0.25) (layer B.Cu) (net 4) (status 800000))
+  (segment (start 195.58 123.825) (end 192.405 120.65) (width 0.25) (layer B.Cu) (net 4))
+  (via (at 195.58 123.825) (size 0.6) (drill 0.4) (layers F.Cu B.Cu) (net 4))
+  (segment (start 186.055 123.825) (end 195.58 123.825) (width 0.25) (layer F.Cu) (net 4))
+  (via (at 186.055 123.825) (size 0.6) (drill 0.4) (layers F.Cu B.Cu) (net 4))
+  (segment (start 182.245 120.015) (end 186.055 123.825) (width 0.25) (layer B.Cu) (net 4))
+  (segment (start 192.405 114.935) (end 192.405 119.38) (width 0.25) (layer B.Cu) (net 4))
+  (segment (start 189.865 112.395) (end 192.405 114.935) (width 0.25) (layer B.Cu) (net 4))
+  (segment (start 186.055 112.395) (end 189.865 112.395) (width 0.25) (layer B.Cu) (net 4))
+  (segment (start 192.405 129.54) (end 192.405 123.825) (width 0.25) (layer B.Cu) (net 5))
+  (segment (start 187.96 114.935) (end 186.055 114.935) (width 0.25) (layer B.Cu) (net 5))
+  (segment (start 189.23 116.205) (end 187.96 114.935) (width 0.25) (layer B.Cu) (net 5))
+  (segment (start 189.23 120.65) (end 189.23 116.205) (width 0.25) (layer B.Cu) (net 5))
+  (segment (start 192.405 123.825) (end 189.23 120.65) (width 0.25) (layer B.Cu) (net 5))
+  (segment (start 172.085 129.54) (end 192.405 129.54) (width 0.25) (layer B.Cu) (net 5))
+  (segment (start 177.165 127) (end 177.165 125.73) (width 0.25) (layer B.Cu) (net 6))
+  (segment (start 176.53 117.475) (end 178.435 117.475) (width 0.25) (layer B.Cu) (net 6))
+  (segment (start 175.26 118.745) (end 176.53 117.475) (width 0.25) (layer B.Cu) (net 6))
+  (segment (start 175.26 123.825) (end 175.26 118.745) (width 0.25) (layer B.Cu) (net 6))
+  (segment (start 177.165 125.73) (end 175.26 123.825) (width 0.25) (layer B.Cu) (net 6))
 )
